File: Hardware/Schematic/Despro2/Despro2.kicad_sch (KiCad schematic)
At the start: 0 parts

Commit message: Schematic Revision
Other:
- added sheet GPIO_Pinout (GPIO_Pinout.kicad_sch)
- sheet MCU ports: added GPIO20, GPIO21, GPIO9; removed none
- sheet Motor Driver ports: added none; removed EnB, IN3, IN4
