File: Hardware/Schematic/Despro2/MCU.kicad_sch (KiCad schematic)
At the start: 7 parts, among them J6 Conn_01x08_Pin, J7 Conn_01x08_Pin, U3 ESP32C3-SUPERMINI

Commit message: Schematic Revision
Changed lines of the file:
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@@
-		)
-	)
-	(label "GPIO9"
-		(at 46.99 46.99 180)
-		(effects
-			(font
-				(size 1.27 1.27)
-			)
-			(justify right bottom)
 		)
 	)
@@
 		)
 	)
-	(label "GPIO20"
-		(at 46.99 52.07 180)
-		(effects
-			(font
-				(size 1.27 1.27)
-			)
-			(justify right bottom)
-		)
-	)
 	(label "GND"
 		(at 106.68 76.2 0)
@@
 		)
 	)
-	(label "GPIO21"
-		(at 46.99 54.61 180)
-		(effects
-			(font
-				(size 1.27 1.27)
-			)
-			(justify right bottom)
-		)
-	)
 	(label "GPIO6"
 		(at 81.28 76.2 180)
@@
 		)
 	)
+	(hierarchical_label "GPIO21"
+		(shape input)
+		(at 46.99 54.61 180)
+		(effects
+			(font
+				(size 1.27 1.27)
+			)
+			(justify right)
+		)
+	)
 	(hierarchical_label "GPIO4"
 		(shape input)
@@
 		)
 	)
+	(hierarchical_label "GPIO20"
+		(shape input)
+		(at 46.99 52.07 180)
+		(effects
+			(font
+				(size 1.27 1.27)
+			)
+			(justify right)
+		)
+	)
 	(hierarchical_label "GPIO10"
 		(shape input)
@@
 		(effects
 			(font
+				(size 1.27 1.27)
+			)
+			(justify right)
+		)
+	)
+	(hierarchical_label "GPIO9"
+		(shape input)
+		(at 46.99 46.99 180)
+		(effects
+			(font
