File: Hardware/Schematic/Despro2/Despro2.kicad_pcb (KiCad board)
At the start: 2 copper layers, 122.8 x 97.2 mm, 43 parts, among them J3 Screw_Terminal_01x04, J4 Screw_Terminal_01x02, J5 Screw_Terminal_01x04, J6 Conn_01x08_Pin, J7 Conn_01x08_Pin, J8 Screw_Terminal_01x02, SW1 SW_SPST, U2 XL4015, U3 ESP32C3-SUPERMINI, U4 L298N

Commit message: SMD variation PCB
Parts:
- added C20: 10u, Capacitor_THT:C_Disc_D5.0mm_W2.5mm_P5.00mm, F.Cu at (173.5, 80.8)
- added J1: Screw_Terminal_01x03, TerminalBlock_Phoenix:TerminalBlock_Phoenix_PT-1,5-3-3.5-H_1x03_P3.50mm_Horizontal, F.Cu at (185.2, 24.3)
- added J10: Buzzer, Connector_Molex:Molex_SL_171971-0002_1x02_P2.54mm_Vertical, F.Cu at (226.8, 96.5)
- added J2: GPS, Connector_Molex:Molex_SL_171971-0004_1x04_P2.54mm_Vertical, F.Cu at (236.7, 94.8)
- added J9: LCD, Connector_Molex:Molex_SL_171971-0004_1x04_P2.54mm_Vertical, F.Cu at (253.2, 97.1)
- added R18: 10k, Resistor_THT:R_Axial_DIN0411_L9.9mm_D3.6mm_P12.70mm_Horizontal, F.Cu at (182.0, 64.9)
- added SW2: SW_SPST, Button_Switch_THT:SW_PUSH_6mm, F.Cu at (168.2, 86.5)
Connections:
- U4 pad 10: /MCU/GPIO7 -> Net-(J1-Pin_3)
- U4 pad 11: /MCU/GPIO8 -> Net-(J1-Pin_1)
- U4 pad 12: /MCU/GPIO6 -> Net-(J1-Pin_2)
Routing:
- net +3.3V: track 6.31 -> 104.6 mm
- net /MCU/GPIO6: track 110.4 -> 37.3 mm
- net /MCU/GPIO8: track 113.3 -> 47.6 mm, vias 0 -> 2
- net +5V: track 205.6 -> 244.0 mm
- net /MCU/GPIO9: track 6.30 -> 43.4 mm, vias 0 -> 2
- net /MCU/GPIO21: track 6.30 -> 28.5 mm, vias 0 -> 2
- net /MCU/GPIO20: track 6.30 -> 25.4 mm, vias 0 -> 2
- net /MCU/GPIO7: track 100.1 -> 83.4 mm, vias 1 -> 4
